File: linemixer2.sch (EAGLE design)
At the start: 82 parts, among them IC1 OPA2134P, IC2 OPA2134P, IC3 OPA2134P, IC4 OPA2134P, IC5 OPA2134P, J1 POWER_JACK

Commit message: rev D
Parts:
- added U$3: DP_LOGO, myparts:DP_LOGO
Other:
- note added: "Rev D"
- note removed: "Rev C"
Changed lines of the file:
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@@
 <part name="R38" library="adafruit" deviceset="R-US_" device="0204/5" value="100k"/>
 <part name="R39" library="adafruit" deviceset="R-US_" device="0204/5" value="100k"/>
+<part name="U$3" library="myparts" deviceset="DP_LOGO" device=""/>
 </parts>
 <sheets>
@@
 <text x="2.54" y="238.76" size="2.54" layer="91">4-Channel Active Line Mixer</text>
 <text x="2.54" y="223.52" size="1.778" layer="91">Andrew Duhan</text>
-<text x="2.54" y="236.22" size="1.778" layer="91">Rev C</text>
+<text x="2.54" y="236.22" size="1.778" layer="91">Rev D</text>
 <text x="2.54" y="226.06" size="1.778" layer="91">2017-06-19</text>
 <text x="2.54" y="121.92" size="1.778" layer="91">Jacks</text>
@@
 <instance part="R38" gate="G$1" x="15.24" y="139.7" rot="R90"/>
 <instance part="R39" gate="G$1" x="15.24" y="175.26" rot="R90"/>
+<instance part="U$3" gate="G$1" x="33.02" y="228.6"/>
 </instances>
 <busses>
